File: PCB/Wheelchair/Wheelchair.kicad_sch (KiCad schematic)
At the start: 22 parts, among them J1 Conn_01x04_Socket, J2 10118193-0001LF, J3 10118193-0001LF, SW1 SW_MEC_5E, U1 MC14069UBCPG, U2 CP2102N-A02-GQFN20

Commit message: PCB_Layout
Parts:
- added J4: Conn_01x06_Pin, Connector_PinHeader_2.54mm:PinHeader_1x06_P2.54mm_Vertical, symbol Connector:Conn_01x06_Pin
- added J5: Conn_01x09_Pin, Connector_PinHeader_2.54mm:PinHeader_1x09_P2.54mm_Vertical, symbol Connector:Conn_01x09_Pin
- A1: footprint PCM_arduino-library:Arduino_Nano_Every_Socket -> arduino-library:Arduino_Nano_Every_Socket
- C1: footprint (none) -> Capacitor_THT:CP_Radial_D5.0mm_P2.50mm
- C2: footprint (none) -> Capacitor_THT:C_Disc_D3.8mm_W2.6mm_P2.50mm
- D1, D2, D3: footprint (none) -> Diode_THT:D_DO-35_SOD27_P7.62mm_Horizontal
- D4, D5, D6: footprint (none) -> LED_THT:LED_D5.0mm
- J1: footprint (none) -> Connector_PinSocket_2.54mm:PinSocket_1x04_P2.54mm_Vertical
- J2, J3: footprint CONN_10118193-0001LF_AMP -> Connector_USB:USB_Micro-B_Amphenol_10118193-0001LF_Horizontal
- R1, R2, R3, R4, R5, R6: footprint (none) -> Resistor_THT:R_Axial_DIN0207_L6.3mm_D2.5mm_P10.16mm_Horizontal
- SW1: footprint (none) -> Button_Switch_THT:SW_PUSH_6mm_H4.3mm
- U1: footprint PDIP-14_ONS -> MC14069UBCP:PDIP-14_ONS
- U2: footprint QFN20_CP2102N_SIL -> footprints:QFN20_CP2102N_SIL
Connections:
- net +5V: now also M1.10 (VMOT)
- net GND: now also M1.9 (GND); no longer U1.10 (OUT5), U1.11 (IN5), U1.12 (OUT6), U1.13 (IN6), U1.5 (IN3), U1.6 (OUT3), U1.8 (OUT4), U1.9 (IN4)
- net PWMA: now also A1.D12 (D12_MISO); no longer A1.D10
- net PWMB: now also A1.D11 (D11_MOSI); no longer A1.D9
- net at A1.A2: now also J4.6 (Pin_6)
- net at A1.A3: now also J4.5 (Pin_5)
- net at A1.A4 (A4/SDA): now also J4.4 (Pin_4)
- net at A1.A5 (A5/SCL): now also J4.3 (Pin_3)
- net at A1.A6: now also J4.2 (Pin_2)
- net at A1.A7: now also J4.1 (Pin_1)
- net at A1.D2: now also J5.9 (Pin_9)
- net at A1.D3: now also J5.8 (Pin_8)
- net at A1.D4: now also J5.7 (Pin_7)
- net at A1.D5: now also J5.6 (Pin_6)
- net at A1.D6: now also J5.5 (Pin_5)
- net at A1.D7: now also J5.4 (Pin_4)
- net at A1.D8: now also J5.3 (Pin_3)
- new net: A1.D10, J5.1 (Pin_1)
- new net: A1.D9, J5.2 (Pin_2)
- no-connect marks 9 -> 22

Commit message: PCB_routed
Parts:
- removed SW1: SW_MEC_5E, Button_Switch_THT:SW_PUSH_6mm_H4.3mm, symbol Switch:SW_MEC_5E
- added SW2: SW_Push_Open_Dual, Button_Switch_THT:SW_PUSH_6mm_H4.3mm, symbol Switch:SW_Push_Open_Dual
Connections:
- net at A1.RST1 (RESET): now also SW2.2
- net at A1.RST2 (RESET): now also SW2.1
Changed lines of the file:
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@@
 	)
 	(no_connect
-		(at 109.22 88.9)
-	)
-	(no_connect
 		(at 224.79 97.79)
 	)
@@
 	)
 	(no_connect
+		(at 111.76 88.9)
+	)
+	(no_connect
+		(at 111.76 78.74)
+	)
+	(no_connect
 		(at 236.22 43.18)
 	)
@@
 	)
 	(no_connect
-		(at 109.22 78.74)
-	)
-	(no_connect
 		(at 236.22 40.64)
 	)
@@
 	(wire
 		(pts
-			(xy 101.6 78.74) (xy 106.68 78.74)
-		)
-		(stroke
-			(width 0)
-			(type default)
-		)
-	)
-	(wire
-		(pts
 			(xy 247.65 134.62) (xy 247.65 137.16)
 		)
@@
 	(wire
 		(pts
-			(xy 101.6 85.09) (xy 101.6 88.9)
+			(xy 160.02 73.66) (xy 160.02 82.55)
 		)
 		(stroke
@@
 	(wire
 		(pts
-			(xy 160.02 73.66) (xy 160.02 82.55)
+			(xy 171.45 88.9) (xy 179.07 88.9)
 		)
 		(stroke
@@
 	(wire
 		(pts
-			(xy 171.45 88.9) (xy 179.07 88.9)
+			(xy 170.18 91.44) (xy 175.26 91.44)
 		)
 		(stroke
@@
 	(wire
 		(pts
-			(xy 170.18 91.44) (xy 175.26 91.44)
+			(xy 101.6 78.74) (xy 106.68 78.74)
 		)
 		(stroke
@@
 	(wire
 		(pts
-			(xy 101.6 82.55) (xy 101.6 78.74)
+			(xy 240.03 147.32) (xy 240.03 151.13)
 		)
 		(stroke
@@
 	(wire
 		(pts
-			(xy 240.03 147.32) (xy 240.03 151.13)
+			(xy 240.03 132.08) (xy 247.65 132.08)
 		)
 		(stroke
@@
 	(wire
 		(pts
-			(xy 240.03 132.08) (xy 247.65 132.08)
+			(xy 101.6 88.9) (xy 106.68 88.9)
 		)
 		(stroke
@@
 	(wire
 		(pts
-			(xy 101.6 88.9) (xy 106.68 88.9)
+			(xy 101.6 82.55) (xy 101.6 78.74)
 		)
 		(stroke
@@
 	(wire
 		(pts
+			(xy 101.6 85.09) (xy 101.6 88.9)
+		)
+		(stroke
+			(width 0)
+			(type default)
+		)
+	)
+	(wire
+		(pts
 			(xy 162.56 105.41) (xy 162.56 99.06)
 		)
@@
 	)
 	(symbol
+		(lib_id "Switch:SW_Push_Open_Dual")
+		(at 106.68 83.82 90)
+		(unit 1)
+		(exclude_from_sim no)
+		(in_bom yes)
+		(on_board yes)
+		(dnp no)
+		(fields_autoplaced yes)
+		(property "Reference" "SW2"
+			(at 114.3 82.5499 90)
+			(effects
+				(font
+					(size 1.27 1.27)
+				)
+				(justify right)
+			)
+		)
+		(property "Value" "SW_Push_Open_Dual"
+			(at 114.3 85.0899 90)
+			(effects
+				(font
+					(size 1.27 1.27)
+				)
+				(justify right)
+			)
+		)
+		(property "Footprint" "Button_Switch_THT:SW_PUSH_6mm_H4.3mm"
+			(at 101.6 83.82 0)
+			(effects
+				(font
+					(size 1.27 1.27)
+				)
+				(hide yes)
+			)
+		)
+		(property "Datasheet" "~"
+			(at 101.6 83.82 0)
+			(effects
+				(font
+					(size 1.27 1.27)
+				)
+				(hide yes)
+			)
+		)
+		(property "Description" "Push button switch, normally closed, generic, four pins"
+			(at 106.68 83.82 0)
+			(effects
+				(font
+					(size 1.27 1.27)
+				)
+				(hide yes)
+			)
+		)
+		(pin "3"
+		)
+		(pin "1"
+		)
+		(pin "4"
+		)
+		(pin "2"
+		)
+		(instances
+			(project ""
+				(path "/44a16fae-3888-4f4d-83db-6d86bd4d2df5"
+					(reference "SW2")
+					(unit 1)
+				)
+			)
+		)
+	)
+	(symbol
 		(lib_id "Device:LED")
 		(at 240.03 143.51 90)
@@
 					(unit 1)
 				)
-			)
-		)
-	)
-	(symbol
-		(lib_id "Switch:SW_MEC_5E")
-		(at 106.68 83.82 270)
-		(unit 1)
-		(exclude_from_sim no)
-		(in_bom yes)
-		(on_board yes)
-		(dnp no)
-		(fields_autoplaced yes)
-		(property "Reference" "SW1"
-			(at 113.03 82.5499 90)
-			(effects
-				(font
-					(size 1.27 1.27)
-				)
-				(justify left)
-			)
-		)
-		(property "Value" "SW_MEC_5E"
-			(at 113.03 85.0899 90)
-			(effects
-				(font
-					(size 1.27 1.27)
-				)
-				(justify left)
-			)
-		)
-		(property "Footprint" "Button_Switch_THT:SW_PUSH_6mm_H4.3mm"
-			(at 114.3 83.82 0)
-			(effects
-				(font
-					(size 1.27 1.27)
-				)
-				(hide yes)
-			)
-		)
-		(property "Datasheet" "http://www.apem.com/int/index.php?controller=attachment&id_attachment=1371"
-			(at 114.3 83.82 0)
-			(effects
-				(font
-					(size 1.27 1.27)
-				)
-				(hide yes)
-			)
-		)
-		(property "Description" "MEC 5E single pole normally-open tactile switch"
-			(at 106.68 83.82 0)
-			(effects
-				(font
-					(size 1.27 1.27)
-				)
-				(hide yes)
-			)
-		)
-		(pin "2"
-		)
-		(pin "3"
-		)
-		(pin "1"
-		)
-		(pin "4"
-		)
-		(instances
-			(project ""
-				(path "/44a16fae-3888-4f4d-83db-6d86bd4d2df5"
-					(reference "SW1")
-					(unit 1)
-				)
